Commit message: fix: urdf
- increase range of m4 (elbow)
- increase collision boundary

File: my_robot/ros2/src/prep_bot/urdf/robot.urdf (robot description, URDF)
Before this commit: robot prep_bot, 9 links, 8 joints
Links:
- link gripper_left: geometry collision box size=0.005 0.03 0.02; visual box size=0.00382 0.015 0.014456
- link gripper_right: geometry collision box size=0.005 0.03 0.02; visual box size=0.00382 0.015 0.014456
Joints:
- joint elbow_joint: limit lower=-1.57 upper=1.57 effort=50 velocity=1.0 -> lower=-2.61 upper=2.61 effort=50 velocity=1.0
- joint gripper_left_joint: limit lower=0 upper=0.02 effort=10 velocity=0.05 -> lower=0 upper=0.0225 effort=10 velocity=0.05; origin xyz=0.01191 0 0.137737 rpy=0 0 0 -> xyz=0.01591 0 0.137737 rpy=0 0 0
- joint gripper_right_joint: limit lower=-0.02 upper=0 effort=10 velocity=0.05 -> lower=-0.0225 upper=0 effort=10 velocity=0.05; origin xyz=0.00809 0 0.137737 rpy=0 0 0 -> xyz=0.00409 0 0.137737 rpy=0 0 0
